File: sebuspill.kicad_pcb (KiCad board)
At the start: 2 copper layers, 67 x 26 mm, 32 parts, among them J1 Conn_01x04_Male, J2 USB_B_Micro, J3 Pinout 1, J4 Pinout 2, U1 AMS1117-3.3, U2 STM32F103C8T6, Y1 16MHz

Commit message: ordered at JLCPCP
Parts:
- SW1: renamed from  
- moved R2 0.81 mm to (146.4, 95.2), turned to 90 degrees
- renumbered D1 to D2
Routing:
- net PC13: track 68.8 -> 58.7 mm
- net +3V3: track 206.0 -> 208.5 mm, vias 12 -> 13
- net GND: track 44.6 -> 46.0 mm, vias 18 -> 77
- net /BOOTP_SW: track 16.9 -> 17.9 mm
- net /BOOT0: track 23.2 -> 22.7 mm
- added copper zone on F.Cu, net GND
- removed copper zone on F.Cu, net +3V3
